File: MRCS-8xDPDT-Relay.brd (EAGLE design)
At the start: 150 x 70 mm, 19 parts, among them CON1 CONNECTOR-M10LOCK, K1 RELAY-G2R2, K2 RELAY-G2R2, K3 RELAY-G2R2, K4 RELAY-G2R2, K5 RELAY-G2R2, K6 RELAY-G2R2, K7 RELAY-G2R2, K8 RELAY-G2R2

Commit message: early doodling
Parts:
- added RELAY_PWR: CONNECTOR-M03MOLEX-254-LOCK, SPCoast:MOLEX-1X3_LOCK
- IC1: value (none) -> ULN2830
- moved CON1 2.54 mm to (57.1, 7.62)
Connections:
- new net +5V: CON1.1, CON2.1, CON4.2, RELAY_PWR.1
- new net N$1: CON1.9, IC1.1
- new net N$10: IC1.16, K3.1
- new net N$11: IC1.15, K4.1
- new net N$12: IC1.14, K5.1
- new net N$13: IC1.18, K1.2
- new net N$14: IC1.13, K6.1
- new net N$15: IC1.12, K7.1
- new net N$16: IC1.11, K8.1
- new net N$17: IC1.10, K1.1, K2.2, K3.2, K4.2, K5.2, K6.2, K7.2, K8.2, RELAY_PWR.2
- new net N$18: J1.1, K1.S1
- new net N$19: J1.2, K1.O1
- new net N$2: CON1.8, IC1.2
- new net N$20: J1.3, K1.P1
- new net N$21: J1.4, K1.S2
- new net N$22: J1.5, K1.O2
- new net N$23: J1.6, K1.P2
- new net N$24: J2.1, K2.S1
- new net N$25: J2.2, K2.O1
- new net N$27: J2.3, K2.P1
- new net N$3: CON1.7, IC1.3
- new net N$4: CON1.6, IC1.4
- new net N$5: CON1.5, IC1.5
- new net N$6: CON1.4, IC1.6
- new net N$7: CON1.3, IC1.7
- new net N$8: CON1.2, IC1.8
- new net N$9: IC1.17, K2.1
- new net VIN: CON3.2, RELAY_PWR.3
- net GND: now also CON1.10, CON2.2, CON2.3, CON3.1, CON4.1
Changed lines of the file:
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@@
 </autorouter>
 <elements>
-<element name="CON1" library="SPCoast" package="1X10_LOCK" value="CONNECTOR-M10LOCK" x="59.69" y="7.62"/>
+<element name="CON1" library="SPCoast" package="1X10_LOCK" value="CONNECTOR-M10LOCK" x="57.15" y="7.62"/>
 <element name="K1" library="SPCoast" package="G2R2" value="RELAY-G2R2" x="17.145" y="40.64" rot="R90">
 <attribute name="MF" value="OMRON COMPONENTS USA" x="17.145" y="40.64" size="1.778" layer="27" font="vector" ratio="10" rot="R90" display="off"/>
@@
 <attribute name="OC_FARNELL" value="unknown" x="132.715" y="40.64" size="1.778" layer="27" font="vector" ratio="10" rot="R90" display="off"/>
 </element>
-<element name="IC1" library="MRCS" package="DIL18" value="" x="69.85" y="17.78"/>
+<element name="IC1" library="MRCS" package="DIL18" value="ULN2830" x="69.85" y="17.78"/>
 <element name="J1" library="SPCoast" package="1X08_LOCK" value="" x="16.51" y="63.5"/>
 <element name="J2" library="SPCoast" package="1X08_LOCK" value="" x="36.83" y="63.5"/>
@@
 <element name="CON3" library="SPCoast" package="SCREWTERMINAL-3.5MM-2_LOCK" value="" x="33.02" y="10.16"/>
 <element name="CON4" library="SPCoast" package="SCREWTERMINAL-3.5MM-2_LOCK" value="" x="104.14" y="8.89"/>
+<element name="RELAY_PWR" library="SPCoast" package="MOLEX-1X3_LOCK" value="CONNECTOR-M03MOLEX-254-LOCK" x="1.27" y="-25.4"/>
 </elements>
 <signals>
 <signal name="GND">
 <contactref element="IC1" pad="9"/>
+<contactref element="CON1" pad="10"/>
+<contactref element="CON4" pad="1"/>
+<contactref element="CON3" pad="1"/>
+<contactref element="CON2" pad="3"/>
+<contactref element="CON2" pad="2"/>
+<wire x1="80.01" y1="7.493" x2="103.9622" y2="8.89" width="0" layer="19" extent="1-1"/>
+<wire x1="80.01" y1="13.97" x2="80.01" y2="7.493" width="0" layer="19" extent="1-1"/>
+<wire x1="32.8422" y1="10.16" x2="80.01" y2="7.493" width="0" layer="19" extent="1-1"/>
+<wire x1="20.0025" y1="11.43" x2="32.8422" y2="10.16" width="0" layer="19" extent="1-1"/>
+<wire x1="15.24" y1="8.255" x2="20.0025" y2="11.43" width="0" layer="19" extent="1-1"/>
+</signal>
+<signal name="N$1">
+<contactref element="CON1" pad="9"/>
+<contactref element="IC1" pad="1"/>
+<wire x1="59.69" y1="13.97" x2="77.47" y2="7.747" width="0" layer="19" extent="1-1"/>
+</signal>
+<signal name="N$2">
+<contactref element="CON1" pad="8"/>
+<contactref element="IC1" pad="2"/>
+<wire x1="62.23" y1="13.97" x2="74.93" y2="7.493" width="0" layer="19" extent="1-1"/>
+</signal>
+<signal name="N$3">
+<contactref element="CON1" pad="7"/>
+<contactref element="IC1" pad="3"/>
+<wire x1="64.77" y1="13.97" x2="72.39" y2="7.747" width="0" layer="19" extent="1-1"/>
+</signal>
+<signal name="N$4">
+<contactref element="CON1" pad="6"/>
+<contactref element="IC1" pad="4"/>
+<wire x1="69.85" y1="7.493" x2="67.31" y2="13.97" width="0" layer="19" extent="1-1"/>
+</signal>
+<signal name="N$5">
+<contactref element="CON1" pad="5"/>
+<contactref element="IC1" pad="5"/>
+<wire x1="67.31" y1="7.747" x2="69.85" y2="13.97" width="0" layer="19" extent="1-1"/>
+</signal>
+<signal name="N$6">
+<contactref element="CON1" pad="4"/>
+<contactref element="IC1" pad="6"/>
+<wire x1="64.77" y1="7.493" x2="72.39" y2="13.97" width="0" layer="19" extent="1-1"/>
+</signal>
+<signal name="N$7">
+<contactref element="CON1" pad="3"/>
+<contactref element="IC1" pad="7"/>
+<wire x1="62.23" y1="7.747" x2="74.93" y2="13.97" width="0" layer="19" extent="1-1"/>
+</signal>
+<signal name="N$8">
+<contactref element="CON1" pad="2"/>
+<contactref element="IC1" pad="8"/>
+<wire x1="59.69" y1="7.493" x2="77.47" y2="13.97" width="0" layer="19" extent="1-1"/>
+</signal>
+<signal name="+5V">
+<contactref element="CON4" pad="2"/>
+<contactref element="CON1" pad="1"/>
+<contactref element="CON2" pad="1"/>
+<contactref element="RELAY_PWR" pad="1"/>
+<wire x1="57.15" y1="7.747" x2="107.8178" y2="8.89" width="0" layer="19" extent="1-1"/>
+<wire x1="15.24" y1="14.605" x2="57.15" y2="7.747" width="0" layer="19" extent="1-1"/>
+<wire x1="1.27" y1="-25.273" x2="15.24" y2="14.605" width="0" layer="19" extent="1-1"/>
+</signal>
+<signal name="VIN">
+<contactref element="CON3" pad="2"/>
+<contactref element="RELAY_PWR" pad="3"/>
+<wire x1="6.35" y1="-25.273" x2="36.6978" y2="10.16" width="0" layer="19" extent="1-1"/>
+</signal>
+<signal name="N$13">
+<contactref element="K1" pad="2"/>
+<contactref element="IC1" pad="18"/>
+<wire x1="13.335" y1="29.21" x2="59.69" y2="21.59" width="0" layer="19" extent="1-1"/>
+</signal>
+<signal name="N$9">
+<contactref element="IC1" pad="17"/>
+<contactref element="K2" pad="1"/>
+<wire x1="37.338" y1="29.21" x2="62.23" y2="21.59" width="0" layer="19" extent="1-1"/>
+</signal>
+<signal name="N$10">
+<contactref element="IC1" pad="16"/>
+<contactref element="K3" pad="1"/>
+<wire x1="53.848" y1="29.21" x2="64.77" y2="21.59" width="0" layer="19" extent="1-1"/>
+</signal>
+<signal name="N$11">
+<contactref element="IC1" pad="15"/>
+<contactref element="K4" pad="1"/>
+<wire x1="67.31" y1="21.59" x2="70.358" y2="29.21" width="0" layer="19" extent="1-1"/>
+</signal>
+<signal name="N$12">
+<contactref element="IC1" pad="14"/>
+<contactref element="K5" pad="1"/>
+<wire x1="69.85" y1="21.59" x2="86.868" y2="29.21" width="0" layer="19" extent="1-1"/>
+</signal>
+<signal name="N$14">
+<contactref element="IC1" pad="13"/>
+<contactref element="K6" pad="1"/>
+<wire x1="72.39" y1="21.59" x2="103.378" y2="29.21" width="0" layer="19" extent="1-1"/>
+</signal>
+<signal name="N$15">
+<contactref element="IC1" pad="12"/>
+<contactref element="K7" pad="1"/>
+<wire x1="74.93" y1="21.59" x2="119.888" y2="29.21" width="0" layer="19" extent="1-1"/>
+</signal>
+<signal name="N$16">
+<contactref element="IC1" pad="11"/>
+<contactref element="K8" pad="1"/>
+<wire x1="77.47" y1="21.59" x2="136.398" y2="29.21" width="0" layer="19" extent="1-1"/>
+</signal>
+<signal name="N$17">
+<contactref element="K8" pad="2"/>
+<contactref element="K7" pad="2"/>
+<contactref element="K6" pad="2"/>
+<contactref element="K5" pad="2"/>
+<contactref element="K4" pad="2"/>
+<contactref element="K3" pad="2"/>
+<contactref element="K2" pad="2"/>
+<contactref element="K1" pad="1"/>
+<contactref element="RELAY_PWR" pad="2"/>
+<contactref element="IC1" pad="10"/>
+<wire x1="112.395" y1="29.21" x2="128.905" y2="29.21" width="0" layer="19" extent="1-1"/>
+<wire x1="95.885" y1="29.21" x2="112.395" y2="29.21" width="0" layer="19" extent="1-1"/>
+<wire x1="79.375" y1="29.21" x2="95.885" y2="29.21" width="0" layer="19" extent="1-1"/>
+<wire x1="80.01" y1="21.59" x2="79.375" y2="29.21" width="0" layer="19" extent="1-1"/>
+<wire x1="62.865" y1="29.21" x2="79.375" y2="29.21" width="0" layer="19" extent="1-1"/>
+<wire x1="46.355" y1="29.21" x2="62.865" y2="29.21" width="0" layer="19" extent="1-1"/>
+<wire x1="29.845" y1="29.21" x2="46.355" y2="29.21" width="0" layer="19" extent="1-1"/>
+<wire x1="20.828" y1="29.21" x2="29.845" y2="29.21" width="0" layer="19" extent="1-1"/>
+<wire x1="3.81" y1="-25.527" x2="20.828" y2="29.21" width="0" layer="19" extent="1-1"/>
+</signal>
+<signal name="N$18">
+<contactref element="K1" pad="S1"/>
+<contactref element="J1" pad="1"/>
+<wire x1="20.828" y1="54.2036" x2="16.51" y2="63.627" width="0" layer="19" extent="1-1"/>
+</signal>
+<signal name="N$19">
+<contactref element="K1" pad="O1"/>
+<contactref element="J1" pad="2"/>
+<wire x1="20.828" y1="44.2214" x2="19.05" y2="63.373" width="0" layer="19" extent="1-1"/>
+</signal>
+<signal name="N$20">
+<contactref element="K1" pad="P1"/>
+<contactref element="J1" pad="3"/>
+<wire x1="20.828" y1="49.1998" x2="21.59" y2="63.627" width="0" layer="19" extent="1-1"/>
+</signal>
+<signal name="N$21">
+<contactref element="J1" pad="4"/>
+<contactref element="K1" pad="S2"/>
+<wire x1="13.335" y1="54.2036" x2="24.13" y2="63.373" width="0" layer="19" extent="1-1"/>
+</signal>
+<signal name="N$22">
+<contactref element="K1" pad="O2"/>
+<contactref element="J1" pad="5"/>
+<wire x1="13.335" y1="44.2214" x2="26.67" y2="63.627" width="0" layer="19" extent="1-1"/>
+</signal>
+<signal name="N$23">
+<contactref element="K1" pad="P2"/>
+<contactref element="J1" pad="6"/>
+<wire x1="13.335" y1="49.1998" x2="29.21" y2="63.373" width="0" layer="19" extent="1-1"/>
+</signal>
+<signal name="N$24">
+<contactref element="J2" pad="1"/>
+<contactref element="K2" pad="S1"/>
+<wire x1="37.338" y1="54.2036" x2="36.83" y2="63.627" width="0" layer="19" extent="1-1"/>
+</signal>
+<signal name="N$25">
+<contactref element="J2" pad="2"/>
+<contactref element="K2" pad="O1"/>
+<wire x1="37.338" y1="44.2214" x2="39.37" y2="63.373" width="0" layer="19" extent="1-1"/>
+</signal>
+<signal name="N$27">
+<contactref element="J2" pad="3"/>
+<contactref element="K2" pad="P1"/>
+<wire x1="37.338" y1="49.1998" x2="41.91" y2="63.627" width="0" layer="19" extent="1-1"/>
 </signal>
 </signals>

Commit message: keeping Jon up to date
adding contacts
Connections:
- new net N$26: J2.1, K2.P1
- new net N$28: J2.3, K2.O2
- new net N$29: J2.4, K2.P2
- new net N$30: J2.7, K3.P2
- new net N$31: J2.6, K3.O2
- new net N$32: J2.8, K3.S1
- new net N$33: J2.5, K3.S2
- new net N$34: J3.1, K3.O1
- new net N$35: J3.2, K3.P1
- new net N$36: J3.3, K4.S1
- new net N$37: J3.4, K4.O1
- new net N$38: J3.5, K4.P1
- new net N$39: J3.6, K4.S2
- new net N$40: J3.7, K4.O2
- new net N$41: J3.8, K4.P2
- net N$24: now also J1.7; no longer J2.1
- net N$25: now also J1.8; no longer J2.2
- net N$27: now also J2.2, K2.S2; no longer J2.3, K2.P1
Changed lines of the file:
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@@
 </signal>
 <signal name="N$24">
-<contactref element="J2" pad="1"/>
 <contactref element="K2" pad="S1"/>
-<wire x1="37.338" y1="54.2036" x2="36.83" y2="63.627" width="0" layer="19" extent="1-1"/>
+<contactref element="J1" pad="7"/>
+<wire x1="37.338" y1="54.2036" x2="31.75" y2="63.627" width="0" layer="19" extent="1-1"/>
 </signal>
 <signal name="N$25">
-<contactref element="J2" pad="2"/>
 <contactref element="K2" pad="O1"/>
-<wire x1="37.338" y1="44.2214" x2="39.37" y2="63.373" width="0" layer="19" extent="1-1"/>
+<contactref element="J1" pad="8"/>
+<wire x1="37.338" y1="44.2214" x2="34.29" y2="63.373" width="0" layer="19" extent="1-1"/>
+</signal>
+<signal name="N$26">
+<contactref element="K2" pad="P1"/>
+<contactref element="J2" pad="1"/>
+<wire x1="37.338" y1="49.1998" x2="36.83" y2="63.627" width="0" layer="19" extent="1-1"/>
 </signal>
 <signal name="N$27">
+<contactref element="K2" pad="S2"/>
+<contactref element="J2" pad="2"/>
+<wire x1="29.845" y1="54.2036" x2="39.37" y2="63.373" width="0" layer="19" extent="1-1"/>
+</signal>
+<signal name="N$28">
+<contactref element="K2" pad="O2"/>
 <contactref element="J2" pad="3"/>
-<contactref element="K2" pad="P1"/>
-<wire x1="37.338" y1="49.1998" x2="41.91" y2="63.627" width="0" layer="19" extent="1-1"/>
+<wire x1="29.845" y1="44.2214" x2="41.91" y2="63.627" width="0" layer="19" extent="1-1"/>
+</signal>
+<signal name="N$29">
+<contactref element="K2" pad="P2"/>
+<contactref element="J2" pad="4"/>
+<wire x1="29.845" y1="49.1998" x2="44.45" y2="63.373" width="0" layer="19" extent="1-1"/>
+</signal>
+<signal name="N$31">
+<contactref element="K3" pad="O2"/>
+<contactref element="J2" pad="6"/>
+<wire x1="46.355" y1="44.2214" x2="49.53" y2="63.373" width="0" layer="19" extent="1-1"/>
+</signal>
+<signal name="N$33">
+<contactref element="J2" pad="5"/>
+<contactref element="K3" pad="S2"/>
+<wire x1="46.355" y1="54.2036" x2="46.99" y2="63.627" width="0" layer="19" extent="1-1"/>
+</signal>
+<signal name="N$30">
+<contactref element="J2" pad="7"/>
+<contactref element="K3" pad="P2"/>
+<wire x1="46.355" y1="49.1998" x2="52.07" y2="63.627" width="0" layer="19" extent="1-1"/>
+</signal>
+<signal name="N$32">
+<contactref element="J2" pad="8"/>
+<contactref element="K3" pad="S1"/>
+<wire x1="53.848" y1="54.2036" x2="54.61" y2="63.373" width="0" layer="19" extent="1-1"/>
+</signal>
+<signal name="N$34">
+<contactref element="J3" pad="1"/>
+<contactref element="K3" pad="O1"/>
+<wire x1="53.848" y1="44.2214" x2="57.15" y2="63.627" width="0" layer="19" extent="1-1"/>
+</signal>
+<signal name="N$35">
+<contactref element="K3" pad="P1"/>
+<contactref element="J3" pad="2"/>
+<wire x1="53.848" y1="49.1998" x2="59.69" y2="63.373" width="0" layer="19" extent="1-1"/>
+</signal>
+<signal name="N$36">
+<contactref element="J3" pad="3"/>
+<contactref element="K4" pad="S1"/>
+<wire x1="70.358" y1="54.2036" x2="62.23" y2="63.627" width="0" layer="19" extent="1-1"/>
+</signal>
+<signal name="N$37">
+<contactref element="J3" pad="4"/>
+<contactref element="K4" pad="O1"/>
+<wire x1="70.358" y1="44.2214" x2="64.77" y2="63.373" width="0" layer="19" extent="1-1"/>
+</signal>
+<signal name="N$38">
+<contactref element="K4" pad="P1"/>
+<contactref element="J3" pad="5"/>
+<wire x1="70.358" y1="49.1998" x2="67.31" y2="63.627" width="0" layer="19" extent="1-1"/>
+</signal>
+<signal name="N$39">
+<contactref element="J3" pad="6"/>
+<contactref element="K4" pad="S2"/>
+<wire x1="62.865" y1="54.2036" x2="69.85" y2="63.373" width="0" layer="19" extent="1-1"/>
+</signal>
+<signal name="N$40">
+<contactref element="J3" pad="7"/>
+<contactref element="K4" pad="O2"/>
+<wire x1="62.865" y1="44.2214" x2="72.39" y2="63.627" width="0" layer="19" extent="1-1"/>
+</signal>
+<signal name="N$41">
+<contactref element="K4" pad="P2"/>
+<contactref element="J3" pad="8"/>
+<wire x1="62.865" y1="49.1998" x2="74.93" y2="63.373" width="0" layer="19" extent="1-1"/>
 </signal>
 </signals>

Commit message: 1st pass complete
first pass. no ground or power jumpers.
Parts:
- moved RELAY_PWR 53.9 mm to (31.8, 19.1)
- moved CON1 22.9 mm to (80.0, 7.62), turned to 180 degrees
- moved J1 17.8 mm to (34.3, 63.5), turned to 180 degrees
- moved CON3 12.0 mm to (43.2, 16.5)
- moved CON4 8.52 mm to (100.3, 16.5)
- moved IC1 1.27 mm to (69.8, 16.5)
Connections:
- new net N$42: J5.4, K6.P1
- new net N$43: J5.5, K7.S2
- new net N$44: J5.6, K7.O2
- new net N$45: J5.7, K7.P2
- new net N$46: J5.8, K7.S1
- new net N$47: J6.1, K7.O1
- new net N$48: J6.2, K7.P1
- new net N$49: J6.3, K8.S2
- new net N$50: J6.4, K8.O2
- new net N$51: J6.5, K8.P2
- new net N$52: J6.6, K8.S1
- new net N$53: J6.7, K8.O1
- new net N$54: J6.8, K8.P1
- new net N$55: J5.3, K6.O1
- new net N$56: J5.2, K6.S1
- new net N$57: J5.1, K6.P2
- new net N$58: J4.8, K6.O2
- new net N$59: J4.7, K6.S2
- new net N$60: J4.6, K5.P1
- new net N$61: J4.5, K5.O1
- new net N$62: J4.4, K5.S1
- new net N$64: J4.2, K5.O2
- new net N$65: J4.1, K5.S2
- new net N$66: J1.4, K1.O1
- net N$13: now also K1.1; no longer K1.2
- net N$17: now also K1.2; no longer K1.1
- net N$18: now also J1.8, K1.S2; no longer J1.1, K1.S1
- net N$19: now also J1.7, K1.O2; no longer J1.2, K1.O1
- net N$21: now also J1.5, K1.S1; no longer J1.4, K1.S2
- net N$22: now also J2.3, K2.O1; no longer J1.5, K1.O2
- net N$24: now also J1.2, K2.S2; no longer J1.7, K2.S1
- net N$25: now also J1.1, K2.O2; no longer J1.8, K2.O1
- net N$26: now also K2.P2; no longer K2.P1
- net N$27: now also K2.S1; no longer K2.S2
- net N$28: now also J4.3, K5.P2; no longer J2.3, K2.O2
- net N$29: now also K2.P1; no longer K2.P2
- net N$36: now also K4.S2; no longer K4.S1
- net N$37: now also K4.O2; no longer K4.O1
- net N$38: now also K4.P2; no longer K4.P1
- net N$39: now also K4.S1; no longer K4.S2
- net N$40: now also K4.O1; no longer K4.O2
- net N$41: now also K4.P1; no longer K4.P2
Routing:
- net N$17: track 0.00 -> 164.6 mm
- net +5V: track 0.00 -> 116.4 mm
- net N$16: track 0.00 -> 66.5 mm
- net N$15: track 0.00 -> 52.2 mm
- net N$13: track 0.00 -> 45.5 mm
- net N$19: track 0.00 -> 38.8 mm
- net N$14: track 0.00 -> 38.2 mm
- net N$9: track 0.00 -> 31.8 mm
- net N$53: track 0.00 -> 27.7 mm
- net N$50: track 0.00 -> 24.8 mm
- net N$44: track 0.00 -> 24.3 mm
- net N$47: track 0.00 -> 23.9 mm
- net N$12: track 0.00 -> 23.7 mm
- net N$58: track 0.00 -> 23.0 mm
- net N$22: track 0.00 -> 22.4 mm
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- added copper zone on layer 16, net GND
Other:
- board text added: "G + N 5 D V"
- board text added: "G R N L D Y"
- board text added: "G12345678+"
- board text added: "MRCS 8xDPDT Relay V. 1.0 20230104 Seth Neumann"
