File: MRCS-8xDPDT-Relay.sch (EAGLE design)
At the start: 19 parts, among them CON1 CONNECTOR-M10LOCK, K1 RELAY-G2R2, K2 RELAY-G2R2, K3 RELAY-G2R2, K4 RELAY-G2R2, K5 RELAY-G2R2, K6 RELAY-G2R2, K7 RELAY-G2R2, K8 RELAY-G2R2

Commit message: early doodling
Parts:
- added RELAY_PWR: CONNECTOR-M03MOLEX-254-LOCK, SPCoast:CONNECTOR-M03MOLEX-254-LOCK
- IC1: value (none) -> ULN2830
Connections:
- new net +5V: CON1.1, CON2.1, CON4.B, RELAY_PWR.1
- new net GND: CON1.10, CON2.2, CON2.3, CON3.A, CON4.A, IC1.GND
- new net N$1: CON1.9, IC1.I1
- new net N$10: IC1.O3, K31.1
- new net N$11: IC1.O4, K41.1
- new net N$12: IC1.O5, K51.1
- new net N$13: IC1.O1, K11.2
- new net N$14: IC1.O6, K61.1
- new net N$15: IC1.O7, K71.1
- new net N$16: IC1.O8, K81.1
- new net N$17: IC1.CD+, K11.1, K21.2, K31.2, K41.2, K51.2, K61.2, K71.2, K81.2, RELAY_PWR.2
- new net N$18: J1.1, K12.S
- new net N$19: J1.2, K12.O
- new net N$2: CON1.8, IC1.I2
- new net N$20: J1.3, K12.P
- new net N$21: J1.4, K13.S
- new net N$22: J1.5, K13.O
- new net N$23: J1.6, K13.P
- new net N$24: J2.1, K22.S
- new net N$25: J2.2, K22.O
- new net N$27: J2.3, K22.P
- new net N$3: CON1.7, IC1.I3
- new net N$4: CON1.6, IC1.I4
- new net N$5: CON1.5, IC1.I5
- new net N$6: CON1.4, IC1.I6
- new net N$7: CON1.3, IC1.I7
- new net N$8: CON1.2, IC1.I8
- new net N$9: IC1.O2, K21.1
- new net VIN: CON3.B, RELAY_PWR.3
Other:
- note added: "GND 8 7 6 5 4 3 2 1 +5"
- note added: "optional relay voltage"
- moved on the sheet: CON1, CON2, CON3, CON4, IC1, J1, J2, J3, J4, J5, J6, K1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

Commit message: keeping Jon up to date
adding contacts
Connections:
- new net N$26: J2.1, K22.P
- new net N$28: J2.3, K23.O
- new net N$29: J2.4, K23.P
- new net N$30: J2.7, K33.P
- new net N$31: J2.6, K33.O
- new net N$32: J2.8, K32.S
- new net N$33: J2.5, K33.S
- new net N$34: J3.1, K32.O
- new net N$35: J3.2, K32.P
- new net N$36: J3.3, K42.S
- new net N$37: J3.4, K42.O
- new net N$38: J3.5, K42.P
- new net N$39: J3.6, K43.S
- new net N$40: J3.7, K43.O
- new net N$41: J3.8, K43.P
- net N$24: now also J1.7; no longer J2.1
- net N$25: now also J1.8; no longer J2.2
- net N$27: now also J2.2, K23.S; no longer J2.3, K22.P
Other:
- moved on the sheet: CON3, J1, J2, J3, J4, J5, J6, K1, K2, K3, K4, K5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

Commit message: 1st pass complete
first pass. no ground or power jumpers.
Connections:
- new net N$42: J5.4, K62.P
- new net N$43: J5.5, K73.S
- new net N$44: J5.6, K73.O
- new net N$45: J5.7, K73.P
- new net N$46: J5.8, K72.S
- new net N$47: J6.1, K72.O
- new net N$48: J6.2, K72.P
- new net N$49: J6.3, K83.S
- new net N$50: J6.4, K83.O
- new net N$51: J6.5, K83.P
- new net N$52: J6.6, K82.S
- new net N$53: J6.7, K82.O
- new net N$54: J6.8, K82.P
- new net N$55: J5.3, K62.O
- new net N$56: J5.2, K62.S
- new net N$57: J5.1, K63.P
- new net N$58: J4.8, K63.O
- new net N$59: J4.7, K63.S
- new net N$60: J4.6, K52.P
- new net N$61: J4.5, K52.O
- new net N$62: J4.4, K52.S
- new net N$64: J4.2, K53.O
- new net N$65: J4.1, K53.S
- new net N$66: J1.4, K12.O
- net N$13: now also K11.1; no longer K11.2
- net N$17: now also K11.2; no longer K11.1
- net N$18: now also J1.8, K13.S; no longer J1.1, K12.S
- net N$19: now also J1.7, K13.O; no longer J1.2, K12.O
- net N$21: now also J1.5, K12.S; no longer J1.4, K13.S
- net N$22: now also J2.3, K22.O; no longer J1.5, K13.O
- net N$24: now also J1.2, K23.S; no longer J1.7, K22.S
- net N$25: now also J1.1, K23.O; no longer J1.8, K22.O
- net N$26: now also K23.P; no longer K22.P
- net N$27: now also K22.S; no longer K23.S
- net N$28: now also J4.3, K53.P; no longer J2.3, K23.O
- net N$29: now also K22.P; no longer K23.P
- net N$36: now also K43.S; no longer K42.S
- net N$37: now also K43.O; no longer K42.O
- net N$38: now also K43.P; no longer K42.P
- net N$39: now also K42.S; no longer K43.S
- net N$40: now also K42.O; no longer K43.O
- net N$41: now also K42.P; no longer K43.P
Other:
- moved on the sheet: CON3, J1, J2, J3, J4, J5, J6, K1, K2, K3, K4, K5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
