File: MRCS-8xDPDT-Relay v1_2.brd (EAGLE design)
At the start: 150 x 70 mm, 39 parts, among them CON3 CONNECTOR-M10LOCK, CON5 CONNECTOR-M03MOLEX-254-LOCK, IC1 ULN2830, K1 G5V-2, K2 G5V-2, K3 G5V-2, K4 G5V-2, K5 G5V-2, K6 G5V-2, K7 G5V-2, K8 G5V-2

Commit message: changes for V1.2
1 - changed polarity of relay so polarized relays will work
2 - Moved the second contact to a separate bus, so you can put any signal you want in by leaving the resistor uncut or cut it and use the contact independently
3 - added connector for bus above, cleaned up labels
Parts:
- added CON6: (no value), SPCoast:SCREWTERMINAL-3.5MM-2_LOCK
- moved CON1 5.08 mm to (48.3, 16.5)
- moved CON5 4.58 mm to (35.6, 16.5)
Connections:
- new net AUX_COMMON: CON6.2, R10.P2, R12.P2, R14.P2, R16.P2, R2.P2, R4.P2, R6.P2, R8.P2
- net GND: now also CON6.1
- net N$10: now also K3.16; no longer K3.1
- net N$11: now also K4.16; no longer K4.1
- net N$12: now also K5.16; no longer K5.1
- net N$14: now also K6.16; no longer K6.1
- net N$15: now also K7.16; no longer K7.1
- net N$16: now also K8.16; no longer K8.1
- net N$22: now also K1.16; no longer K1.1
- net N$9: now also K2.16; no longer K2.1
- net RELAY_POWER: now also K1.1, K2.1, K3.1, K4.1, K5.1, K6.1, K7.1, K8.1; no longer K1.16, K2.16, K3.16, K4.16, K5.16, K6.16, K7.16, K8.16, R10.P2, R12.P2, R14.P2, R16.P2, R2.P2, R4.P2, R6.P2, R8.P2
Routing:
- net AUX_COMMON: track 0.00 -> 201.3 mm, vias 0 -> 1
- net RELAY_POWER: track 337.1 -> 219.1 mm
- net N$22: track 50.6 -> 58.7 mm
- net N$14: track 42.2 -> 34.6 mm
- net N$12: track 30.6 -> 23.0 mm
- net N$9: track 37.9 -> 45.5 mm
- net N$10: track 25.2 -> 32.8 mm
- net N$15: track 55.7 -> 48.0 mm
- net N$16: track 66.9 -> 60.0 mm
- net +5V: track 119.7 -> 112.9 mm
- net N$11: track 17.6 -> 20.5 mm
- net VIN: track 11.2 -> 13.5 mm
Other:
- board text added: "5 R R V E L L Y"
- board text added: "G A N U D X"
- board text added: "MRCS 8xDPDT Relay V. 1.2 20230402 Seth Neumann"
- board text removed: "MRCS 8xDPDT Relay V. 1.1 20230125 Seth Neumann"
